File: electronics/8dof/forcefoot.sch (EAGLE design)
At the start: 108 parts

Commit message: Adding clock, tweaking placing
Parts:
- added C33, C34, C35, C36, C37, C38, C39, C40: 20pF, SparkFun-Passives:CAP0805
- added R47: ?, rhoban:RESISTANCE-R0805
Connections:
- net 5A+ renamed 6A+
- removed net 5A-: C20.1, HX5.IN_A-, R39.1, R40.2, U$14.3
- new net CLOCK: C33.2, C34.2, C35.2, C36.2, C37.2, C38.2, C39.2, C40.2, MAPLE_MINI.8, R47.2
- new net N$16: C33.1, HX1.X1
- new net N$17: C34.1, HX5.X1
- new net N$18: C35.1, HX6.X1
- new net N$19: C36.1, HX7.X1
- new net N$20: C37.1, HX8.X1
- new net N$21: C38.1, HX4.X1
- new net N$22: C39.1, HX3.X1
- new net N$23: C40.1, HX2.X1
- net 5BASE: now also HX6.BASE, U$17.B; no longer HX5.BASE, U$11.B
- net 6A-: now also C20.1, HX5.IN_A-, R39.1, R40.2, U$14.3
- net 6BASE: now also HX5.BASE, U$11.B; no longer HX6.BASE, U$17.B
- net 7A-: now also C32.1, HX8.IN_A-, U$22.3; no longer C28.1, HX7.IN_A-, U$20.3
- net 7BASE: now also HX8.BASE, U$21.B; no longer HX7.BASE, U$19.B
- net 8A-: now also C28.1, HX7.IN_A-, U$20.3; no longer C32.1, HX8.IN_A-, U$22.3
- net 8BASE: now also HX7.BASE, U$19.B; no longer HX8.BASE, U$21.B
- net AVDD$5: now also C23.2, HX6.AVDD, R28.2, R41.2, U$17.C, U$18.2; no longer C19.2, HX5.AVDD, R37.2, R39.2, U$11.C, U$14.2
- net AVDD$6: now also C19.2, HX5.AVDD, R37.2, R39.2, U$11.C, U$14.2; no longer C23.2, HX6.AVDD, R28.2, R41.2, U$17.C, U$18.2
- net AVDD$7: now also C31.2, HX8.AVDD, R34.2, R45.2, U$21.C, U$22.2; no longer C27.2, HX7.AVDD, R31.2, R43.2, U$19.C, U$20.2
- net AVDD$8: now also C27.2, HX7.AVDD, R31.2, R43.2, U$19.C, U$20.2; no longer C31.2, HX8.AVDD, R34.2, R45.2, U$21.C, U$22.2
- net DOUT2: now also MAPLE_MINI.19; no longer MAPLE_MINI.18
- net DOUT3: now also MAPLE_MINI.21; no longer MAPLE_MINI.24
- net DOUT4: now also MAPLE_MINI.23; no longer MAPLE_MINI.26
- net DOUT5: now also HX6.DOUT, MAPLE_MINI.25; no longer HX5.DOUT, MAPLE_MINI.20
- net DOUT6: now also HX5.DOUT, MAPLE_MINI.27; no longer HX6.DOUT, MAPLE_MINI.22
- net DOUT7: now also HX8.DOUT, MAPLE_MINI.29; no longer HX7.DOUT, MAPLE_MINI.28
- net DOUT8: now also HX7.DOUT, MAPLE_MINI.31; no longer HX8.DOUT, MAPLE_MINI.30
- net GND: now also R47.1; no longer HX1.X1, HX2.X1, HX3.X1, HX4.X1, HX5.X1, HX6.X1, HX7.X1, HX8.X1
- net SCK2: now also MAPLE_MINI.18; no longer MAPLE_MINI.31
- net SCK3: now also MAPLE_MINI.20; no longer MAPLE_MINI.23
- net SCK4: now also MAPLE_MINI.22; no longer MAPLE_MINI.25
- net SCK5: now also HX6.SCK, MAPLE_MINI.24; no longer HX5.SCK, MAPLE_MINI.19
- net SCK6: now also HX5.SCK, MAPLE_MINI.26; no longer HX6.SCK, MAPLE_MINI.21
- net SCK7: now also HX8.SCK, MAPLE_MINI.28; no longer HX7.SCK, MAPLE_MINI.27
- net SCK8: now also HX7.SCK, MAPLE_MINI.30; no longer HX8.SCK, MAPLE_MINI.29
Other:
- moved on the sheet: C1, C13, C17, C18, C19, C20, C21, C22, C23, C24, C25, C26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

Commit message: Using 1.5mm 4p connectors
Parts:
- U$10, U$13, U$14, U$18, U$20, U$22, U$3, U$7: value CONNEC_1X04" -> CONNEC_1X041.5; device rhoban:CONNEC_1X04" -> rhoban:CONNEC_1X041.5
Changed lines of the file:
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@@
 <part name="GND14" library="supply1" deviceset="GND" device=""/>
 <part name="U$23" library="rhoban" deviceset="CONNEC_1X03" device=""/>
-<part name="U$3" library="rhoban" deviceset="CONNEC_1X04" device="&quot;"/>
-<part name="U$7" library="rhoban" deviceset="CONNEC_1X04" device="&quot;"/>
-<part name="U$10" library="rhoban" deviceset="CONNEC_1X04" device="&quot;"/>
-<part name="U$13" library="rhoban" deviceset="CONNEC_1X04" device="&quot;"/>
-<part name="U$14" library="rhoban" deviceset="CONNEC_1X04" device="&quot;"/>
-<part name="U$18" library="rhoban" deviceset="CONNEC_1X04" device="&quot;"/>
-<part name="U$20" library="rhoban" deviceset="CONNEC_1X04" device="&quot;"/>
-<part name="U$22" library="rhoban" deviceset="CONNEC_1X04" device="&quot;"/>
+<part name="U$3" library="rhoban" deviceset="CONNEC_1X04" device="1.5"/>
+<part name="U$7" library="rhoban" deviceset="CONNEC_1X04" device="1.5"/>
+<part name="U$10" library="rhoban" deviceset="CONNEC_1X04" device="1.5"/>
+<part name="U$13" library="rhoban" deviceset="CONNEC_1X04" device="1.5"/>
+<part name="U$14" library="rhoban" deviceset="CONNEC_1X04" device="1.5"/>
+<part name="U$18" library="rhoban" deviceset="CONNEC_1X04" device="1.5"/>
+<part name="U$20" library="rhoban" deviceset="CONNEC_1X04" device="1.5"/>
+<part name="U$22" library="rhoban" deviceset="CONNEC_1X04" device="1.5"/>
 <part name="GND15" library="supply1" deviceset="GND" device=""/>
 <part name="GND16" library="supply1" deviceset="GND" device=""/>

Commit message: Tying B-/B+ to ground
Connections:
- net GND: now also HX1.IN_B+, HX1.IN_B-, HX2.IN_B+, HX2.IN_B-, HX3.IN_B+, HX3.IN_B-, HX4.IN_B+, HX4.IN_B-, HX5.IN_B+, HX5.IN_B-, HX6.IN_B+, HX6.IN_B-, HX7.IN_B+, HX7.IN_B-, HX8.IN_B+, HX8.IN_B-
Changed lines of the file:
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@@
 <part name="C39" library="SparkFun-Passives" deviceset="CAP" device="0805" value="20pF"/>
 <part name="C40" library="SparkFun-Passives" deviceset="CAP" device="0805" value="20pF"/>
+<part name="GND9" library="supply1" deviceset="GND" device=""/>
+<part name="GND24" library="supply1" deviceset="GND" device=""/>
+<part name="GND25" library="supply1" deviceset="GND" device=""/>
+<part name="GND26" library="supply1" deviceset="GND" device=""/>
+<part name="GND27" library="supply1" deviceset="GND" device=""/>
+<part name="GND28" library="supply1" deviceset="GND" device=""/>
+<part name="GND29" library="supply1" deviceset="GND" device=""/>
+<part name="GND30" library="supply1" deviceset="GND" device=""/>
 </parts>
 <sheets>
@@
 <instance part="C39" gate="G$1" x="342.9" y="58.42" rot="R90"/>
 <instance part="C40" gate="G$1" x="223.52" y="58.42" rot="R90"/>
+<instance part="GND9" gate="1" x="55.88" y="35.56"/>
+<instance part="GND24" gate="1" x="175.26" y="33.02"/>
+<instance part="GND25" gate="1" x="294.64" y="33.02"/>
+<instance part="GND26" gate="1" x="408.94" y="33.02"/>
+<instance part="GND27" gate="1" x="406.4" y="-60.96"/>
+<instance part="GND28" gate="1" x="279.4" y="-66.04"/>
+<instance part="GND29" gate="1" x="157.48" y="-66.04"/>
+<instance part="GND30" gate="1" x="38.1" y="-60.96"/>
 </instances>
 <busses>
@@
 <pinref part="GND23" gate="1" pin="GND"/>
 </segment>
+<segment>
+<pinref part="HX1" gate="G$1" pin="IN_B-"/>
+<pinref part="HX1" gate="G$1" pin="IN_B+"/>
+<wire x1="55.88" y1="43.18" x2="55.88" y2="40.64" width="0.1524" layer="91"/>
+<wire x1="55.88" y1="38.1" x2="55.88" y2="40.64" width="0.1524" layer="91"/>
+<pinref part="GND9" gate="1" pin="GND"/>
+<junction x="55.88" y="40.64"/>
+<junction x="55.88" y="43.18"/>
+</segment>
+<segment>
+<wire x1="175.26" y1="40.64" x2="175.26" y2="38.1" width="0.1524" layer="91"/>
+<wire x1="175.26" y1="35.56" x2="175.26" y2="38.1" width="0.1524" layer="91"/>
+<pinref part="GND24" gate="1" pin="GND"/>
+<pinref part="HX2" gate="G$1" pin="IN_B+"/>
+<junction x="175.26" y="38.1"/>
+<pinref part="HX2" gate="G$1" pin="IN_B-"/>
+<junction x="175.26" y="40.64"/>
+</segment>
+<segment>
+<wire x1="294.64" y1="40.64" x2="294.64" y2="38.1" width="0.1524" layer="91"/>
+<wire x1="294.64" y1="35.56" x2="294.64" y2="38.1" width="0.1524" layer="91"/>
+<pinref part="GND25" gate="1" pin="GND"/>
+<pinref part="HX3" gate="G$1" pin="IN_B+"/>
+<junction x="294.64" y="38.1"/>
+<pinref part="HX3" gate="G$1" pin="IN_B-"/>
+<junction x="294.64" y="40.64"/>
+</segment>
+<segment>
+<wire x1="408.94" y1="40.64" x2="408.94" y2="38.1" width="0.1524" layer="91"/>
+<wire x1="408.94" y1="35.56" x2="408.94" y2="38.1" width="0.1524" layer="91"/>
+<pinref part="GND26" gate="1" pin="GND"/>
+<pinref part="HX4" gate="G$1" pin="IN_B+"/>
+<junction x="408.94" y="38.1"/>
+<pinref part="HX4" gate="G$1" pin="IN_B-"/>
+<junction x="408.94" y="40.64"/>
+</segment>
+<segment>
+<wire x1="406.4" y1="-53.34" x2="406.4" y2="-55.88" width="0.1524" layer="91"/>
+<wire x1="406.4" y1="-58.42" x2="406.4" y2="-55.88" width="0.1524" layer="91"/>
+<pinref part="GND27" gate="1" pin="GND"/>
+<pinref part="HX7" gate="G$1" pin="IN_B+"/>
+<junction x="406.4" y="-55.88"/>
+<pinref part="HX7" gate="G$1" pin="IN_B-"/>
+<junction x="406.4" y="-53.34"/>
+</segment>
+<segment>
+<wire x1="279.4" y1="-58.42" x2="279.4" y2="-60.96" width="0.1524" layer="91"/>
+<wire x1="279.4" y1="-63.5" x2="279.4" y2="-60.96" width="0.1524" layer="91"/>
+<pinref part="GND28" gate="1" pin="GND"/>
+<pinref part="HX8" gate="G$1" pin="IN_B+"/>
+<junction x="279.4" y="-60.96"/>
+<pinref part="HX8" gate="G$1" pin="IN_B-"/>
+<junction x="279.4" y="-58.42"/>
+</segment>
+<segment>
+<wire x1="157.48" y1="-58.42" x2="157.48" y2="-60.96" width="0.1524" layer="91"/>
+<wire x1="157.48" y1="-63.5" x2="157.48" y2="-60.96" width="0.1524" layer="91"/>
+<pinref part="GND29" gate="1" pin="GND"/>
+<pinref part="HX5" gate="G$1" pin="IN_B+"/>
+<junction x="157.48" y="-60.96"/>
+<pinref part="HX5" gate="G$1" pin="IN_B-"/>
+<junction x="157.48" y="-58.42"/>
+</segment>
+<segment>
+<wire x1="38.1" y1="-53.34" x2="38.1" y2="-55.88" width="0.1524" layer="91"/>
+<wire x1="38.1" y1="-58.42" x2="38.1" y2="-55.88" width="0.1524" layer="91"/>
+<pinref part="GND30" gate="1" pin="GND"/>
+<pinref part="HX6" gate="G$1" pin="IN_B+"/>
+<junction x="38.1" y="-55.88"/>
+<pinref part="HX6" gate="G$1" pin="IN_B-"/>
+<junction x="38.1" y="-53.34"/>
+</segment>
 </net>

Commit message: Update schema
Connections:
- removed net 1A-4: R41.1, R42.2
- removed net N$15: U$18.3
- new net 5A-: C24.1, HX6.IN_A-, R41.1, R42.2, U$18.3
- net 6A-: no longer C24.1, HX6.IN_A-
Changed lines of the file:
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@@
-</segment>
-</net>
-<net name="1A-4" class="0">
-<segment>
-<wire x1="7.62" y1="-68.58" x2="-10.16" y2="-68.58" width="0.1524" layer="91"/>
-<pinref part="R41" gate="G$1" pin="1"/>
-<pinref part="R42" gate="G$1" pin="2"/>
-<junction x="-10.16" y="-68.58"/>
 </segment>
 </net>
@@
 </net>
 <net name="6A-" class="0">
-<segment>
-<pinref part="HX6" gate="G$1" pin="IN_A-"/>
-<pinref part="C24" gate="G$1" pin="1"/>
-<wire x1="38.1" y1="-48.26" x2="27.94" y2="-48.26" width="0.1524" layer="91"/>
-<wire x1="27.94" y1="-48.26" x2="27.94" y2="-71.12" width="0.1524" layer="91"/>
-</segment>
 <segment>
 <wire x1="127" y1="-83.82" x2="116.84" y2="-83.82" width="0.1524" layer="91"/>
@@
 </segment>
 </net>
-<net name="N$15" class="0">
-<segment>
-<wire x1="7.62" y1="-78.74" x2="7.62" y2="-68.58" width="0.1524" layer="91"/>
-<wire x1="7.62" y1="-78.74" x2="-2.54" y2="-78.74" width="0.1524" layer="91"/>
-<label x="10.16" y="-68.58" size="1.778" layer="95"/>
-<pinref part="U$18" gate="G$1" pin="3"/>
-</segment>
-</net>
 <net name="CLOCK" class="0">
 <segment>
@@
 </segment>
 </net>
+<net name="5A-" class="0">
+<segment>
+<pinref part="R41" gate="G$1" pin="1"/>
+<pinref part="R42" gate="G$1" pin="2"/>
+<junction x="-10.16" y="-68.58"/>
+<pinref part="HX6" gate="G$1" pin="IN_A-"/>
+<pinref part="C24" gate="G$1" pin="1"/>
+<wire x1="38.1" y1="-48.26" x2="27.94" y2="-48.26" width="0.1524" layer="91"/>
+<wire x1="27.94" y1="-48.26" x2="27.94" y2="-68.58" width="0.1524" layer="91"/>
+<wire x1="27.94" y1="-68.58" x2="27.94" y2="-71.12" width="0.1524" layer="91"/>
+<wire x1="-10.16" y1="-68.58" x2="7.62" y2="-68.58" width="0.1524" layer="91"/>
+<label x="15.24" y="-71.12" size="1.778" layer="95"/>
+<wire x1="7.62" y1="-68.58" x2="27.94" y2="-68.58" width="0.1524" layer="91"/>
+<wire x1="7.62" y1="-78.74" x2="7.62" y2="-68.58" width="0.1524" layer="91"/>
+<wire x1="7.62" y1="-78.74" x2="-2.54" y2="-78.74" width="0.1524" layer="91"/>
+<pinref part="U$18" gate="G$1" pin="3"/>
+<junction x="7.62" y="-68.58"/>
+</segment>
+</net>

Commit message: Fixes
Connections:
- removed net 1A-1: R21.1, R22.2
- removed net 1A-2: R23.1, R24.2
- removed net 1A-3: R25.1, R26.2
- removed net 1A-5: R43.1, R44.2
- removed net 1A-6: R45.1, R46.2
- net 2A-: now also R21.1, R22.2
- net 3A-: now also R23.1, R24.2
- net 4A-: now also R25.1, R26.2
- net 7A-: now also R45.1, R46.2
- net 8A-: now also R43.1, R44.2
- net DIRECTION: now also MAPLE_MINI.3; no longer MAPLE_MINI.2
- net DOUT4: now also MAPLE_MINI.2; no longer MAPLE_MINI.23
- net SCK5: now also MAPLE_MINI.6; no longer MAPLE_MINI.24
Changed lines of the file:
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@@
 </segment>
 <segment>
-<pinref part="MAPLE_MINI" gate="G$1" pin="23"/>
-<wire x1="12.7" y1="132.08" x2="10.16" y2="132.08" width="0.1524" layer="91"/>
-<label x="2.54" y="132.08" size="1.778" layer="95"/>
+<pinref part="MAPLE_MINI" gate="G$1" pin="2"/>
+<wire x1="38.1" y1="119.38" x2="40.64" y2="119.38" width="0.1524" layer="91"/>
+<label x="40.64" y="119.38" size="1.778" layer="95"/>
 </segment>
 </net>
@@
 <junction x="165.1" y="25.4"/>
 <pinref part="U$7" gate="G$1" pin="3"/>
+<wire x1="144.78" y1="25.4" x2="127" y2="25.4" width="0.1524" layer="91"/>
+<pinref part="R21" gate="G$1" pin="1"/>
+<pinref part="R22" gate="G$1" pin="2"/>
+<junction x="127" y="25.4"/>
+<junction x="144.78" y="25.4"/>
 </segment>
 </net>
@@
 <pinref part="U$13" gate="G$1" pin="3"/>
 </segment>
+<segment>
+<wire x1="378.46" y1="25.4" x2="360.68" y2="25.4" width="0.1524" layer="91"/>
+<pinref part="R25" gate="G$1" pin="1"/>
+<pinref part="R26" gate="G$1" pin="2"/>
+<junction x="360.68" y="25.4"/>
+</segment>
 </net>
 <net name="3A-" class="0">
@@
 <junction x="284.48" y="25.4"/>
 <pinref part="U$10" gate="G$1" pin="3"/>
+</segment>
+<segment>
+<wire x1="264.16" y1="25.4" x2="246.38" y2="25.4" width="0.1524" layer="91"/>
+<pinref part="R23" gate="G$1" pin="1"/>
+<pinref part="R24" gate="G$1" pin="2"/>
+<junction x="246.38" y="25.4"/>
 </segment>
 </net>
@@
 </segment>
 <segment>
-<pinref part="MAPLE_MINI" gate="G$1" pin="2"/>
-<wire x1="38.1" y1="119.38" x2="40.64" y2="119.38" width="0.1524" layer="91"/>
-<label x="40.64" y="119.38" size="1.778" layer="95"/>
+<pinref part="MAPLE_MINI" gate="G$1" pin="3"/>
+<wire x1="38.1" y1="121.92" x2="40.64" y2="121.92" width="0.1524" layer="91"/>
+<label x="40.64" y="121.92" size="1.778" layer="95"/>
 </segment>
 </net>
@@
 <wire x1="408.94" y1="71.12" x2="406.4" y2="71.12" width="0.1524" layer="91"/>
 <label x="398.78" y="71.12" size="1.778" layer="95"/>
-</segment>
-</net>
-<net name="1A-1" class="0">
-<segment>
-<wire x1="144.78" y1="25.4" x2="127" y2="25.4" width="0.1524" layer="91"/>
-<pinref part="R21" gate="G$1" pin="1"/>
-<pinref part="R22" gate="G$1" pin="2"/>
-<junction x="127" y="25.4"/>
-</segment>
-</net>
-<net name="1A-2" class="0">
-<segment>
-<wire x1="264.16" y1="25.4" x2="246.38" y2="25.4" width="0.1524" layer="91"/>
-<pinref part="R23" gate="G$1" pin="1"/>
-<pinref part="R24" gate="G$1" pin="2"/>
-<junction x="246.38" y="25.4"/>
-</segment>
-</net>
-<net name="1A-3" class="0">
-<segment>
-<wire x1="378.46" y1="25.4" x2="360.68" y2="25.4" width="0.1524" layer="91"/>
-<pinref part="R25" gate="G$1" pin="1"/>
-<pinref part="R26" gate="G$1" pin="2"/>
-<junction x="360.68" y="25.4"/>
 </segment>
 </net>
@@
 </segment>
 </net>
-<net name="1A-5" class="0">
-<segment>
-<wire x1="375.92" y1="-68.58" x2="358.14" y2="-68.58" width="0.1524" layer="91"/>
-<pinref part="R43" gate="G$1" pin="1"/>
-<pinref part="R44" gate="G$1" pin="2"/>
-<junction x="358.14" y="-68.58"/>
-</segment>
-</net>
-<net name="1A-6" class="0">
-<segment>
-<wire x1="248.92" y1="-73.66" x2="231.14" y2="-73.66" width="0.1524" layer="91"/>
-<pinref part="R45" gate="G$1" pin="1"/>
-<pinref part="R46" gate="G$1" pin="2"/>
-<junction x="231.14" y="-73.66"/>
-</segment>
-</net>
 <net name="SCK5" class="0">
-<segment>
-<pinref part="MAPLE_MINI" gate="G$1" pin="24"/>
-<wire x1="12.7" y1="129.54" x2="10.16" y2="129.54" width="0.1524" layer="91"/>
-<label x="2.54" y="129.54" size="1.778" layer="95"/>
-</segment>
 <segment>
 <pinref part="HX6" gate="G$1" pin="SCK"/>
 <wire x1="78.74" y1="-45.72" x2="81.28" y2="-45.72" width="0.1524" layer="91"/>
 <label x="81.28" y="-45.72" size="1.778" layer="95"/>
+</segment>
+<segment>
+<pinref part="MAPLE_MINI" gate="G$1" pin="6"/>
+<wire x1="38.1" y1="129.54" x2="40.64" y2="129.54" width="0.1524" layer="91"/>
+<label x="40.64" y="129.54" size="1.778" layer="95"/>
 </segment>
 </net>
@@
 <pinref part="U$20" gate="G$1" pin="3"/>
 </segment>
+<segment>
+<wire x1="375.92" y1="-68.58" x2="358.14" y2="-68.58" width="0.1524" layer="91"/>
+<pinref part="R43" gate="G$1" pin="1"/>
+<pinref part="R44" gate="G$1" pin="2"/>
+<junction x="358.14" y="-68.58"/>
+</segment>
 </net>
 <net name="CLOCK" class="0">
@@
 <pinref part="U$22" gate="G$1" pin="3"/>
 </segment>
-</net>
+<segment>
+<wire x1="248.92" y1="-73.66" x2="231.14" y2="-73.66" width="0.1524" layer="91"/>
+<pinref part="R45" gate="G$1" pin="1"/>
+<pinref part="R46" gate="G$1" pin="2"/>
+<junction x="231.14" y="-73.66"/>
+</segment>
+</net>

Commit message: Fix
Connections:
- net DIRECTION: now also MAPLE_MINI.2; no longer MAPLE_MINI.3
- net DOUT4: now also MAPLE_MINI.3; no longer MAPLE_MINI.2
Changed lines of the file:
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@@
 </segment>
 <segment>
-<pinref part="MAPLE_MINI" gate="G$1" pin="2"/>
-<wire x1="38.1" y1="119.38" x2="40.64" y2="119.38" width="0.1524" layer="91"/>
-<label x="40.64" y="119.38" size="1.778" layer="95"/>
+<pinref part="MAPLE_MINI" gate="G$1" pin="3"/>
+<wire x1="38.1" y1="121.92" x2="40.64" y2="121.92" width="0.1524" layer="91"/>
+<label x="40.64" y="121.92" size="1.778" layer="95"/>
 </segment>
 </net>
@@
 </segment>
 <segment>
-<pinref part="MAPLE_MINI" gate="G$1" pin="3"/>
-<wire x1="38.1" y1="121.92" x2="40.64" y2="121.92" width="0.1524" layer="91"/>
-<label x="40.64" y="121.92" size="1.778" layer="95"/>
-</segment>
-</net>
+<pinref part="MAPLE_MINI" gate="G$1" pin="2"/>
+<wire x1="38.1" y1="119.38" x2="40.64" y2="119.38" width="0.1524" layer="91"/>
+<label x="40.64" y="119.38" size="1.778" layer="95"/>
+</segment>
+</net>
