File: electronics/atmega/forcefoot.sch (EAGLE design)
At the start: 68 parts, among them U2 ATMEGA168

Commit message: Fixing pins...
Parts:
- R14, R15: value 3k -> 22
Connections:
- net DOUT4: now also U2.PB1(OC1A); no longer U2.ADC7
- net SCK4: now also U2.PB0(ICP); no longer U2.ADC6
Changed lines of the file:
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@@
 <part name="GND2" library="supply1" deviceset="GND" device=""/>
 <part name="P+1" library="supply1" deviceset="VCC" device=""/>
-<part name="R14" library="rhoban" deviceset="RESISTANCE" device="-R0805" value="3k"/>
-<part name="R15" library="rhoban" deviceset="RESISTANCE" device="-R0805" value="3k"/>
+<part name="R14" library="rhoban" deviceset="RESISTANCE" device="-R0805" value="22"/>
+<part name="R15" library="rhoban" deviceset="RESISTANCE" device="-R0805" value="22"/>
 <part name="R19" library="SparkFun-Passives" deviceset="RESISTOR" device="0805-RES" value="3K"/>
 <part name="R20" library="SparkFun-Passives" deviceset="RESISTOR" device="0805-RES" value="3K"/>
@@
 </segment>
 <segment>
-<wire x1="198.12" y1="160.02" x2="200.66" y2="160.02" width="0.1524" layer="91"/>
-<label x="200.66" y="160.02" size="1.778" layer="95"/>
-<pinref part="U2" gate="G$1" pin="ADC6"/>
+<pinref part="U2" gate="G$1" pin="PB0(ICP)"/>
+<wire x1="198.12" y1="129.54" x2="203.2" y2="129.54" width="0.1524" layer="91"/>
+<label x="203.2" y="129.54" size="1.778" layer="95"/>
 </segment>
 </net>
@@
 </segment>
 <segment>
-<wire x1="198.12" y1="157.48" x2="200.66" y2="157.48" width="0.1524" layer="91"/>
-<label x="200.66" y="157.48" size="1.778" layer="95"/>
-<pinref part="U2" gate="G$1" pin="ADC7"/>
+<pinref part="U2" gate="G$1" pin="PB1(OC1A)"/>
+<wire x1="198.12" y1="127" x2="203.2" y2="127" width="0.1524" layer="91"/>
+<label x="203.2" y="127" size="1.778" layer="95"/>
 </segment>
 </net>

Commit message: Fixes
Connections:
- removed net 1A-1: R21.1, R22.2
- removed net 1A-2: R23.1, R24.2
- removed net 1A-3: R25.1, R26.2
- net 2A-: now also R21.1, R22.2
- net 3A-: now also R23.1, R24.2
- net 4A-: now also R25.1, R26.2
- net VCC: now also R27.2, U$28.2, U2.AREF, U2.VCC@1, U2.VCC@2
- net VIN: no longer R27.2, U$28.2, U2.AREF, U2.VCC@1, U2.VCC@2
Changed lines of the file:
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@@
 <label x="226.06" y="187.96" size="1.778" layer="95"/>
+</segment>
+<segment>
+<pinref part="U$28" gate="G$1" pin="2"/>
+<wire x1="190.5" y1="106.68" x2="193.04" y2="106.68" width="0.1524" layer="91"/>
+<label x="193.04" y="106.68" size="1.778" layer="95"/>
+</segment>
+<segment>
+<wire x1="144.78" y1="187.96" x2="144.78" y2="185.42" width="0.1524" layer="91"/>
+<pinref part="R27" gate="G$1" pin="2"/>
+<label x="144.78" y="187.96" size="1.778" layer="95"/>
+</segment>
+<segment>
+<wire x1="119.38" y1="167.64" x2="119.38" y2="165.1" width="0.1524" layer="91"/>
+<wire x1="119.38" y1="165.1" x2="147.32" y2="165.1" width="0.1524" layer="91"/>
+<wire x1="147.32" y1="165.1" x2="149.86" y2="165.1" width="0.1524" layer="91"/>
+<wire x1="149.86" y1="167.64" x2="147.32" y2="167.64" width="0.1524" layer="91"/>
+<wire x1="147.32" y1="167.64" x2="147.32" y2="165.1" width="0.1524" layer="91"/>
+<junction x="147.32" y="165.1"/>
+<wire x1="149.86" y1="160.02" x2="147.32" y2="160.02" width="0.1524" layer="91"/>
+<wire x1="147.32" y1="160.02" x2="147.32" y2="165.1" width="0.1524" layer="91"/>
+<label x="119.38" y="167.64" size="1.778" layer="95"/>
+<pinref part="U2" gate="G$1" pin="VCC@1"/>
+<pinref part="U2" gate="G$1" pin="VCC@2"/>
+<pinref part="U2" gate="G$1" pin="AREF"/>
 </segment>
 </net>
@@
 <junction x="7.62" y="27.94"/>
 <pinref part="HX1" gate="G$1" pin="IN_A-"/>
+<junction x="25.4" y="27.94"/>
 </segment>
 </net>
@@
 <wire x1="144.78" y1="15.24" x2="144.78" y2="25.4" width="0.1524" layer="91"/>
 <junction x="165.1" y="25.4"/>
+<wire x1="144.78" y1="25.4" x2="127" y2="25.4" width="0.1524" layer="91"/>
+<pinref part="R21" gate="G$1" pin="1"/>
+<pinref part="R22" gate="G$1" pin="2"/>
+<junction x="127" y="25.4"/>
+<junction x="144.78" y="25.4"/>
 </segment>
 </net>
@@
 <wire x1="378.46" y1="15.24" x2="378.46" y2="25.4" width="0.1524" layer="91"/>
 <junction x="398.78" y="25.4"/>
+<wire x1="378.46" y1="25.4" x2="360.68" y2="25.4" width="0.1524" layer="91"/>
+<pinref part="R25" gate="G$1" pin="1"/>
+<pinref part="R26" gate="G$1" pin="2"/>
+<junction x="360.68" y="25.4"/>
+<junction x="378.46" y="25.4"/>
 </segment>
 </net>
@@
 <wire x1="264.16" y1="15.24" x2="264.16" y2="25.4" width="0.1524" layer="91"/>
 <junction x="284.48" y="25.4"/>
+<wire x1="264.16" y1="25.4" x2="246.38" y2="25.4" width="0.1524" layer="91"/>
+<pinref part="R23" gate="G$1" pin="1"/>
+<pinref part="R24" gate="G$1" pin="2"/>
+<junction x="246.38" y="25.4"/>
+<junction x="264.16" y="25.4"/>
 </segment>
 </net>
@@
 <label x="292.1" y="124.46" size="1.778" layer="95"/>
 <pinref part="U$8" gate="G$1" pin="2"/>
-</segment>
-<segment>
-<pinref part="U$28" gate="G$1" pin="2"/>
-<wire x1="190.5" y1="106.68" x2="193.04" y2="106.68" width="0.1524" layer="91"/>
-<label x="193.04" y="106.68" size="1.778" layer="95"/>
-</segment>
-<segment>
-<wire x1="119.38" y1="167.64" x2="119.38" y2="165.1" width="0.1524" layer="91"/>
-<wire x1="119.38" y1="165.1" x2="147.32" y2="165.1" width="0.1524" layer="91"/>
-<wire x1="147.32" y1="165.1" x2="149.86" y2="165.1" width="0.1524" layer="91"/>
-<wire x1="149.86" y1="167.64" x2="147.32" y2="167.64" width="0.1524" layer="91"/>
-<wire x1="147.32" y1="167.64" x2="147.32" y2="165.1" width="0.1524" layer="91"/>
-<junction x="147.32" y="165.1"/>
-<wire x1="149.86" y1="160.02" x2="147.32" y2="160.02" width="0.1524" layer="91"/>
-<wire x1="147.32" y1="160.02" x2="147.32" y2="165.1" width="0.1524" layer="91"/>
-<label x="119.38" y="167.64" size="1.778" layer="95"/>
-<pinref part="U2" gate="G$1" pin="VCC@1"/>
-<pinref part="U2" gate="G$1" pin="VCC@2"/>
-<pinref part="U2" gate="G$1" pin="AREF"/>
-</segment>
-<segment>
-<wire x1="144.78" y1="187.96" x2="144.78" y2="185.42" width="0.1524" layer="91"/>
-<pinref part="R27" gate="G$1" pin="2"/>
-<label x="144.78" y="187.96" size="1.778" layer="95"/>
 </segment>
 <segment>
@@
 </segment>
 </net>
-<net name="1A-1" class="0">
-<segment>
-<wire x1="144.78" y1="25.4" x2="127" y2="25.4" width="0.1524" layer="91"/>
-<pinref part="R21" gate="G$1" pin="1"/>
-<pinref part="R22" gate="G$1" pin="2"/>
-<junction x="127" y="25.4"/>
-</segment>
-</net>
-<net name="1A-2" class="0">
-<segment>
-<wire x1="264.16" y1="25.4" x2="246.38" y2="25.4" width="0.1524" layer="91"/>
-<pinref part="R23" gate="G$1" pin="1"/>
-<pinref part="R24" gate="G$1" pin="2"/>
-<junction x="246.38" y="25.4"/>
-</segment>
-</net>
-<net name="1A-3" class="0">
-<segment>
-<wire x1="378.46" y1="25.4" x2="360.68" y2="25.4" width="0.1524" layer="91"/>
-<pinref part="R25" gate="G$1" pin="1"/>
-<pinref part="R26" gate="G$1" pin="2"/>
-<junction x="360.68" y="25.4"/>
-</segment>
-</net>
