File: electronics/atmega/forcefoot.brd (EAGLE design)
At the start: 60 x 43.6 mm, 71 parts, among them U2 ATMEGA168

Commit message: Fixing pins...
Parts:
- R14, R15: value 3k -> 22
- moved HX1 0.22 mm to (8.90, 12.8)
Connections:
- net DOUT4: now also U2.13; no longer U2.22
- net SCK4: now also U2.12; no longer U2.19
Routing:
- net SCK2: track 17.7 -> 61.6 mm
- net SCK3: track 69.4 -> 34.1 mm
- net DOUT2: track 48.8 -> 19.1 mm, vias 0 -> 2
- net VCC: track 194.7 -> 222.3 mm, vias 3 -> 2
- net RESET: track 25.8 -> 53.3 mm, vias 2 -> 0
- net RX: track 34.3 -> 54.4 mm, vias 2 -> 0
- net MISO: track 21.8 -> 39.2 mm
- net DOUT4: track 36.2 -> 28.4 mm
- net GND: track 310.5 -> 303.7 mm, vias 5 -> 4
- net RS-: track 38.7 -> 32.1 mm, vias 1 -> 2
- net DOUT3: track 35.2 -> 29.9 mm
- net 3BASE: track 4.49 -> 9.01 mm, vias 0 -> 2
- net SCK: track 21.6 -> 17.2 mm
- net VIN: track 65.7 -> 62.0 mm, vias 3 -> 2
- net 2BASE: track 9.12 -> 5.61 mm, vias 2 -> 0
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
Commit message: Board fixes
Parts:
- moved C9 4.11 mm to (34.1, 16.9), turned to 90 degrees
- moved C1 3.82 mm to (2.79, 16.8), turned to 90 degrees
- moved C5 3.68 mm to (16.0, 16.7), turned to 90 degrees
- moved C13 3.57 mm to (47.6, 17.1), turned to 90 degrees
- moved R4 0.90 mm to (19.1, 8.71)
- moved C10 0.90 mm to (41.8, 8.83)
- moved C11 0.90 mm to (34.1, 2.95)
- moved C12 0.90 mm to (44.8, 8.94)
- moved C14 0.90 mm to (55.0, 9.26)
- moved C16 0.90 mm to (57.8, 9.27)
- moved C2 0.90 mm to (9.35, 8.65)
- moved C4 0.90 mm to (12.3, 8.75)
- moved C8 0.90 mm to (25.1, 8.65)
- moved HX3 0.90 mm to (40.5, 13.8)
- moved HX4 0.90 mm to (53.7, 14.0)
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Routing:
- net VCC: track 222.3 -> 176.6 mm
- net DOUT2: track 19.1 -> 57.5 mm
- net RX: track 54.4 -> 32.8 mm, vias 0 -> 2
- net RESET: track 53.3 -> 34.4 mm, vias 0 -> 2
- net MISO: track 39.2 -> 22.1 mm
- net GND: track 303.7 -> 290.0 mm, vias 4 -> 6
- net SCK2: track 61.6 -> 75.3 mm
- net VIN: track 62.0 -> 73.6 mm
- net IMU_SCL: track 23.1 -> 15.1 mm, vias 1 -> 2
- net AVDD$3: track 19.1 -> 26.6 mm
- net RS-: track 32.1 -> 39.0 mm, vias 2 -> 0
- net 3.3: track 12.3 -> 6.25 mm
- net SCK3: track 34.1 -> 28.1 mm
- net SCK: track 17.2 -> 22.9 mm, vias 1 -> 2
- net IMU_SDA: track 16.1 -> 21.4 mm
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
Commit message: Fixes
Connections:
- removed net 1A-1: R21.1, R22.2
- removed net 1A-2: R23.1, R24.2
- removed net 1A-3: R25.1, R26.2
- net 2A-: now also R21.1, R22.2
- net 3A-: now also R23.1, R24.2
- net 4A-: now also R25.1, R26.2
- net VCC: now also R27.2, U$28.2, U2.20, U2.4, U2.6
- net VIN: no longer R27.2, U$28.2, U2.20, U2.4, U2.6
Routing:
- net SCK2: track 75.3 -> 19.1 mm
- net VIN: track 73.6 -> 28.0 mm, vias 2 -> 0
- net GND: track 290.0 -> 313.0 mm, vias 6 -> 3
- net VCC: track 176.6 -> 195.9 mm, vias 2 -> 3
- net DOUT3: track 24.9 -> 39.8 mm
- net 4A-: track 9.68 -> 19.3 mm, vias 0 -> 1
- net RS-: track 39.0 -> 29.9 mm
- net SCK3: track 28.1 -> 37.1 mm
- net 2A-: track 11.1 -> 19.2 mm, vias 0 -> 1
- net 3A-: track 15.0 -> 22.7 mm, vias 0 -> 2
- net AVDD$3: track 26.6 -> 19.1 mm, vias 0 -> 1
- net RESET: track 34.4 -> 26.9 mm
- net N$19: track 12.3 -> 18.8 mm, vias 2 -> 1
- net IMU_SCL: track 15.1 -> 20.8 mm, vias 2 -> 3
- net TX: track 30.7 -> 25.9 mm
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
Commit message: Moving connector
Parts:
- moved U$28 14.0 mm to (46.9, 38.6), turned to 180 degrees
- moved U$2 11.3 mm to (46.5, 27.7), turned to 90 degrees
- moved U$8 2.90 mm to (31.7, 42.9)
Routing:
- net GND: track 313.0 -> 0.00 mm, vias 3 -> 0
- net VCC: track 195.9 -> 0.00 mm, vias 3 -> 0
- net DOUT2: track 54.5 -> 0.00 mm, vias 2 -> 0
- net DOUT1: track 40.5 -> 0.00 mm, vias 2 -> 0
- net DOUT3: track 39.8 -> 0.00 mm, vias 2 -> 0
- net SCK3: track 37.1 -> 0.00 mm, vias 2 -> 0
- net RX: track 32.8 -> 0.00 mm, vias 2 -> 0
- net RS-: track 29.9 -> 0.00 mm
- net SCK1: track 29.8 -> 0.00 mm
- net SCK4: track 29.5 -> 0.00 mm, vias 2 -> 0
- net VIN: track 28.0 -> 0.00 mm
- net RESET: track 26.9 -> 0.00 mm, vias 2 -> 0
- net DIRECTION: track 26.8 -> 0.00 mm, vias 2 -> 0
- net DOUT4: track 26.5 -> 0.00 mm, vias 2 -> 0
- net TX: track 25.9 -> 0.00 mm, vias 2 -> 0
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
Commit message: board
Routing:
- net GND: track 0.00 -> 313.8 mm, vias 0 -> 2
- net VCC: track 0.00 -> 191.1 mm, vias 0 -> 2
- net DOUT2: track 0.00 -> 57.8 mm, vias 0 -> 2
- net MISO: track 0.00 -> 44.5 mm, vias 0 -> 1
- net DOUT1: track 0.00 -> 36.5 mm, vias 0 -> 2
- net SCK3: track 0.00 -> 35.7 mm, vias 0 -> 2
- net RX: track 0.00 -> 31.7 mm, vias 0 -> 2
- net RESET: track 0.00 -> 31.5 mm, vias 0 -> 2
- net SCK: track 0.00 -> 31.2 mm, vias 0 -> 2
- net VIN: track 0.00 -> 30.9 mm
- net SCK4: track 0.00 -> 30.3 mm, vias 0 -> 2
- net SCK1: track 0.00 -> 30.1 mm, vias 0 -> 2
- net MOSI: track 0.00 -> 27.5 mm, vias 0 -> 2
- net DOUT4: track 0.00 -> 27.0 mm, vias 0 -> 2
- net DIRECTION: track 0.00 -> 27.0 mm, vias 0 -> 2
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